Commit message: Added robot to Gazebo, created a control plugin, and created launch files

File: description/robot.urdf.xacro (robot description, xacro)
@@ -2,4 +2,5 @@
 <robot xmlns:xacro="http://www.ros.org/wiki/xacro"  name="robot">
     <!-- Example link -->
-    <xacro:include filename ="robot_core.xacro" />
+    <xacro:include filename="robot_core.xacro" />
+    <xacro:include filename="gazebo_control.xacro"/>
 </robot>

File: description/robot_core.xacro (robot description, xacro)
@@ -41,4 +41,9 @@
         </xacro:inertial_box>
     </link>
+    <gazebo reference="chassis">
+        <material>
+            Gazebo/White
+        </material>
+    </gazebo>
     <!-- LEFT WHEEL LINK -->
     <joint name="left_wheel_joint" type="continuous">
@@ -65,4 +70,9 @@
         </xacro:inertial_cylinder>
     </link>
+    <gazebo reference="left_wheel">
+        <material>
+            Gazebo/Blue
+        </material>
+    </gazebo>
     <!-- Right WHEEL LINK -->
     <joint name="right_wheel_joint" type="continuous">
@@ -89,4 +99,9 @@
         </xacro:inertial_cylinder>
     </link>
+    <gazebo reference="right_wheel">
+        <material>
+            Gazebo/Blue
+        </material>
+    </gazebo>
     <!-- Caster wheel link -->
     <joint name="caster_wheel_joint" type="fixed">
@@ -111,3 +126,11 @@
         </xacro:inertial_sphere>
     </link>
+   <gazebo reference="caster_wheel">
+        <material>
+            Gazebo/Black
+        </material>
+        <!-- set friction to be 0 -->
+        <mu1 value="0.0001"/>
+        <mu2 value="0.0001"/>
+    </gazebo>
 </robot>
